Commit message: 重构程序框架

File: robot_simulation_ws/src/bullet_simulation_pkg/urdf/dexh13_left.urdf (robot description, URDF)
Before this commit: robot dexh13_right, 17 links, 16 joints
Links:
- removed link right_index_link_0
- removed link right_index_link_1
- removed link right_index_link_2
- removed link right_index_link_3
- removed link right_middle_link_0
- removed link right_middle_link_1
- removed link right_middle_link_2
- removed link right_middle_link_3
- removed link right_palm
- removed link right_ring_link_0
- removed link right_ring_link_1
- removed link right_ring_link_2
- removed link right_ring_link_3
- removed link right_thumb_link_0
- removed link right_thumb_link_1
- removed link right_thumb_link_2
- removed link right_thumb_link_3
- added link left_index_link_0, mass 0.000219582291910095; collision mesh filename=package://bullet_simulation_pkg/meshes/dexh13_left/meshes/l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; visual mesh filename=package://bullet_simulation_pkg/meshes/dexh13_left/meshes/l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
- added link left_index_link_1, mass 0.0112425437662123; collision mesh filename=package://bullet_simulation_pkg/meshes/dexh13_left/meshes/l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; visual mesh filename=package://bullet_simulation_pkg/meshes/dexh13_left/meshes/l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
- added link left_index_link_2, mass 0.00609408297717352; collision mesh filename=package://bullet_simulation_pkg/meshes/dexh13_left/meshes/l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; visual mesh filename=package://bullet_simulation_pkg/meshes/dexh13_left/meshes/l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
- added link left_index_link_3, mass 0.00843580676681889; collision mesh filename=package://bullet_simulation_pkg/meshes/dexh13_left/meshes/l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; visual mesh filename=package://bullet_simulation_pkg/meshes/dexh13_left/meshes/l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
- added link left_middle_link_0, mass 0.000219582291910095; collision mesh filename=package://bullet_simulation_pkg/meshes/dexh13_left/meshes/l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; visual mesh filename=package://bullet_simulation_pkg/meshes/dexh13_left/meshes/l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
- added link left_middle_link_1, mass 0.0112425344934482; collision mesh filename=package://bullet_simulation_pkg/meshes/dexh13_left/meshes/l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; visual mesh filename=package://bullet_simulation_pkg/meshes/dexh13_left/meshes/l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
- added link left_middle_link_2, mass 0.00609408297717341; collision mesh filename=package://bullet_simulation_pkg/meshes/dexh13_left/meshes/l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; visual mesh filename=package://bullet_simulation_pkg/meshes/dexh13_left/meshes/l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
- added link left_middle_link_3, mass 0.00843580796640825; collision mesh filename=package://bullet_simulation_pkg/meshes/dexh13_left/meshes/l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; visual mesh filename=package://bullet_simulation_pkg/meshes/dexh13_left/meshes/l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
- added link left_palm, mass 0.14615; collision mesh filename=package://bullet_simulation_pkg/meshes/dexh13_left/meshes/l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; visual mesh filename=package://bullet_simulation_pkg/meshes/dexh13_left/meshes/l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
- added link left_ring_link_0, mass 0.000219582291910096; collision mesh filename=package://bullet_simulation_pkg/meshes/dexh13_left/meshes/l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; visual mesh filename=package://bullet_simulation_pkg/meshes/dexh13_left/meshes/l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
- added link left_ring_link_1, mass 0.0112425427188638; collision mesh filename=package://bullet_simulation_pkg/meshes/dexh13_left/meshes/l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; visual mesh filename=package://bullet_simulation_pkg/meshes/dexh13_left/meshes/l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
- added link left_ring_link_2, mass 0.00609408297717322; collision mesh filename=package://bullet_simulation_pkg/meshes/dexh13_left/meshes/l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; visual mesh filename=package://bullet_simulation_pkg/meshes/dexh13_left/meshes/l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
- added link left_ring_link_3, mass 0.0084358; collision mesh filename=package://bullet_simulation_pkg/meshes/dexh13_left/meshes/l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; visual mesh filename=package://bullet_simulation_pkg/meshes/dexh13_left/meshes/l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
- added link left_thumb_link_0, mass 0.000219582291910095; collision mesh filename=package://bullet_simulation_pkg/meshes/dexh13_left/meshes/l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; visual mesh filename=package://bullet_simulation_pkg/meshes/dexh13_left/meshes/l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
- added link left_thumb_link_1, mass 0.00513633275560094; collision mesh filename=package://bullet_simulation_pkg/meshes/dexh13_left/meshes/l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; visual mesh filename=package://bullet_simulation_pkg/meshes/dexh13_left/meshes/l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
- added link left_thumb_link_2, mass 0.0167101102599617; collision mesh filename=package://bullet_simulation_pkg/meshes/dexh13_left/meshes/l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; visual mesh filename=package://bullet_simulation_pkg/meshes/dexh13_left/meshes/l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
- added link left_thumb_link_3, mass 0.0166230921101523; collision mesh filename=package://bullet_simulation_pkg/meshes/dexh13_left/meshes/l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; visual mesh filename=package://bullet_simulation_pkg/meshes/dexh13_left/meshes/l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
Joints:
- removed joint right_index_joint_0
- removed joint right_index_joint_1
- removed joint right_index_joint_2
- removed joint right_index_joint_3
- removed joint right_middle_joint_0
- removed joint right_middle_joint_1
- removed joint right_middle_joint_2
- removed joint right_middle_joint_3
- removed joint right_ring_joint_0
- removed joint right_ring_joint_1
- removed joint right_ring_joint_2
- removed joint right_ring_joint_3
- removed joint right_thumb_joint_0
- removed joint right_thumb_joint_1
- removed joint right_thumb_joint_2
- removed joint right_thumb_joint_3
- added joint left_index_joint_0: type revolute, parent left_palm, child left_index_link_0, origin xyz=0.122 0.0315 0.00175 rpy=0 0 0, axis 0 0 1, limit lower=-0.349 upper=0.349 effort=1 velocity=2
- added joint left_index_joint_1: type revolute, parent left_index_link_0, child left_index_link_1, origin xyz=0 0 0 rpy=1.5708 0 0, axis 0 0 1, limit lower=0 upper=1.5707 effort=1 velocity=2
- added joint left_index_joint_2: type revolute, parent left_index_link_1, child left_index_link_2, origin xyz=0.04 0 0 rpy=0 0 0, axis 0 0 1, limit lower=0 upper=1.5707 effort=1 velocity=2
- added joint left_index_joint_3: type revolute, parent left_index_link_2, child left_index_link_3, origin xyz=0.03 0 0 rpy=0 0 0, axis 0 0 1, limit lower=0 upper=1.5707 effort=1 velocity=2
- added joint left_middle_joint_0: type revolute, parent left_palm, child left_middle_link_0, origin xyz=0.122 0 0.00175 rpy=0 0 0, axis 0 0 1, limit lower=-0.349 upper=0.349 effort=1 velocity=2
- added joint left_middle_joint_1: type revolute, parent left_middle_link_0, child left_middle_link_1, origin xyz=0 0 0 rpy=1.5708 0 0, axis 0 0 1, limit lower=0 upper=1.5707 effort=1 velocity=2
- added joint left_middle_joint_2: type revolute, parent left_middle_link_1, child left_middle_link_2, origin xyz=0.04 0 0 rpy=0 0 0, axis 0 0 1, limit lower=0 upper=1.5707 effort=1 velocity=2
- added joint left_middle_joint_3: type revolute, parent left_middle_link_2, child left_middle_link_3, origin xyz=0.03 0 0 rpy=0 0 0, axis 0 0 1, limit lower=0 upper=1.5707 effort=1 velocity=2
- added joint left_ring_joint_0: type revolute, parent left_palm, child left_ring_link_0, origin xyz=0.122 -0.0315 0.00175 rpy=0 0 0, axis 0 0 1, limit lower=-0.349 upper=0.349 effort=1 velocity=2
- added joint left_ring_joint_1: type revolute, parent left_ring_link_0, child left_ring_link_1, origin xyz=0 0 0 rpy=1.5708 0 0, axis 0 0 1, limit lower=0 upper=1.5707 effort=1 velocity=2
- added joint left_ring_joint_2: type revolute, parent left_ring_link_1, child left_ring_link_2, origin xyz=0.04 0 0 rpy=0 0 0, axis 0 0 1, limit lower=0 upper=1.5707 effort=1 velocity=2
- added joint left_ring_joint_3: type revolute, parent left_ring_link_2, child left_ring_link_3, origin xyz=0.03 0 0 rpy=0 0 0, axis 0 0 1, limit lower=0 upper=1.5707 effort=1 velocity=2
- added joint left_thumb_joint_0: type revolute, parent left_palm, child left_thumb_link_0, origin xyz=0.026 0.0365 -0.00025 rpy=0 0 1.5708, axis 0 0 1, limit lower=-0.349 upper=0.349 effort=1 velocity=2
- added joint left_thumb_joint_1: type revolute, parent left_thumb_link_0, child left_thumb_link_1, origin xyz=0 0 0 rpy=1.5708 0 0, axis 0 0 1, limit lower=0 upper=1.5707 effort=1 velocity=2
- added joint left_thumb_joint_2: type revolute, parent left_thumb_link_1, child left_thumb_link_2, origin xyz=0.039999 0.009 0.0215 rpy=1.5708 -0.261799388 0, axis 0 0 1, limit lower=0 upper=1.5707 effort=1 velocity=2
- added joint left_thumb_joint_3: type revolute, parent left_thumb_link_2, child left_thumb_link_3, origin xyz=0.063556 -0.017141 0 rpy=0 0 0, axis 0 0 1, limit lower=0 upper=1.5707 effort=1 velocity=2

File: robot_simulation_ws/src/bullet_simulation_pkg/urdf/dexh13_right.urdf (robot description, URDF)
Before this commit: robot dexh13_left, 17 links, 16 joints
Links:
- removed link left_index_link_0
- removed link left_index_link_1
- removed link left_index_link_2
- removed link left_index_link_3
- removed link left_middle_link_0
- removed link left_middle_link_1
- removed link left_middle_link_2
- removed link left_middle_link_3
- removed link left_palm
- removed link left_ring_link_0
- removed link left_ring_link_1
- removed link left_ring_link_2
- removed link left_ring_link_3
- removed link left_thumb_link_0
- removed link left_thumb_link_1
- removed link left_thumb_link_2
- removed link left_thumb_link_3
- added link right_index_link_0, mass 0.00021958; collision mesh filename=package://bullet_simulation_pkg/meshes/dexh13_right/meshes/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; visual mesh filename=package://bullet_simulation_pkg/meshes/dexh13_right/meshes/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
- added link right_index_link_1, mass 0.011243; collision mesh filename=package://bullet_simulation_pkg/meshes/dexh13_right/meshes/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; visual mesh filename=package://bullet_simulation_pkg/meshes/dexh13_right/meshes/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
- added link right_index_link_2, mass 0.0060940829771732; collision mesh filename=package://bullet_simulation_pkg/meshes/dexh13_right/meshes/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; visual mesh filename=package://bullet_simulation_pkg/meshes/dexh13_right/meshes/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
- added link right_index_link_3, mass 0.0084358; collision mesh filename=package://bullet_simulation_pkg/meshes/dexh13_right/meshes/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; visual mesh filename=package://bullet_simulation_pkg/meshes/dexh13_right/meshes/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
- added link right_middle_link_0, mass 0.00021958; collision mesh filename=package://bullet_simulation_pkg/meshes/dexh13_right/meshes/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; visual mesh filename=package://bullet_simulation_pkg/meshes/dexh13_right/meshes/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
- added link right_middle_link_1, mass 0.011243; collision mesh filename=package://bullet_simulation_pkg/meshes/dexh13_right/meshes/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; visual mesh filename=package://bullet_simulation_pkg/meshes/dexh13_right/meshes/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
- added link right_middle_link_2, mass 0.0060941; collision mesh filename=package://bullet_simulation_pkg/meshes/dexh13_right/meshes/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; visual mesh filename=package://bullet_simulation_pkg/meshes/dexh13_right/meshes/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
- added link right_middle_link_3, mass 0.0084358; collision mesh filename=package://bullet_simulation_pkg/meshes/dexh13_right/meshes/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; visual mesh filename=package://bullet_simulation_pkg/meshes/dexh13_right/meshes/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
- added link right_palm, mass 0.14602; collision mesh filename=package://bullet_simulation_pkg/meshes/dexh13_right/meshes/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; visual mesh filename=package://bullet_simulation_pkg/meshes/dexh13_right/meshes/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
- added link right_ring_link_0, mass 0; collision mesh filename=package://bullet_simulation_pkg/meshes/dexh13_right/meshes/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; visual mesh filename=package://bullet_simulation_pkg/meshes/dexh13_right/meshes/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
- added link right_ring_link_1, mass 0.011243; collision mesh filename=package://bullet_simulation_pkg/meshes/dexh13_right/meshes/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; visual mesh filename=package://bullet_simulation_pkg/meshes/dexh13_right/meshes/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
- added link right_ring_link_2, mass 0.0060941; collision mesh filename=package://bullet_simulation_pkg/meshes/dexh13_right/meshes/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; visual mesh filename=package://bullet_simulation_pkg/meshes/dexh13_right/meshes/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
- added link right_ring_link_3, mass 0.0084358; collision mesh filename=package://bullet_simulation_pkg/meshes/dexh13_right/meshes/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; visual mesh filename=package://bullet_simulation_pkg/meshes/dexh13_right/meshes/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
- added link right_thumb_link_0, mass 0.00021958; collision mesh filename=package://bullet_simulation_pkg/meshes/dexh13_right/meshes/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; visual mesh filename=package://bullet_simulation_pkg/meshes/dexh13_right/meshes/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
- added link right_thumb_link_1, mass 0.0051746; collision mesh filename=package://bullet_simulation_pkg/meshes/dexh13_right/meshes/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; visual mesh filename=package://bullet_simulation_pkg/meshes/dexh13_right/meshes/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
- added link right_thumb_link_2, mass 0.0167100811373488; collision mesh filename=package://bullet_simulation_pkg/meshes/dexh13_right/meshes/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; visual mesh filename=package://bullet_simulation_pkg/meshes/dexh13_right/meshes/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
- added link right_thumb_link_3, mass 0.016623; collision mesh filename=package://bullet_simulation_pkg/meshes/dexh13_right/meshes/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; visual mesh filename=package://bullet_simulation_pkg/meshes/dexh13_right/meshes/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
Joints:
- removed joint left_index_joint_0
- removed joint left_index_joint_1
- removed joint left_index_joint_2
- removed joint left_index_joint_3
- removed joint left_middle_joint_0
- removed joint left_middle_joint_1
- removed joint left_middle_joint_2
- removed joint left_middle_joint_3
- removed joint left_ring_joint_0
- removed joint left_ring_joint_1
- removed joint left_ring_joint_2
- removed joint left_ring_joint_3
- removed joint left_thumb_joint_0
- removed joint left_thumb_joint_1
- removed joint left_thumb_joint_2
- removed joint left_thumb_joint_3
- added joint right_index_joint_0: type revolute, parent right_palm, child right_index_link_0, origin xyz=0.122 -0.0315 0.00175 rpy=-3.1416 0 0, axis 0 0 1, limit lower=-0.349 upper=0.349 effort=1 velocity=2
- added joint right_index_joint_1: type revolute, parent right_index_link_0, child right_index_link_1, origin xyz=0 0 0 rpy=-1.5708 0 0, axis 0 0 1, limit lower=0 upper=1.5707 effort=1 velocity=2
- added joint right_index_joint_2: type revolute, parent right_index_link_1, child right_index_link_2, origin xyz=0.04 0 0 rpy=0 0 0, axis 0 0 1, limit lower=0 upper=1.5707 effort=1 velocity=2
- added joint right_index_joint_3: type revolute, parent right_index_link_2, child right_index_link_3, origin xyz=0.03 0 0 rpy=0 0 0, axis 0 0 1, limit lower=0 upper=1.5707 effort=1 velocity=2
- added joint right_middle_joint_0: type revolute, parent right_palm, child right_middle_link_0, origin xyz=0.122 0 0.00175 rpy=-3.1416 0 0, axis 0 0 1, limit lower=-0.349 upper=0.349 effort=1 velocity=2
- added joint right_middle_joint_1: type revolute, parent right_middle_link_0, child right_middle_link_1, origin xyz=0 0 0 rpy=-1.5708 0 0, axis 0 0 1, limit lower=0 upper=1.5707 effort=1 velocity=2
- added joint right_middle_joint_2: type revolute, parent right_middle_link_1, child right_middle_link_2, origin xyz=0.04 0 0 rpy=0 0 0, axis 0 0 1, limit lower=0 upper=1.5707 effort=1 velocity=2
- added joint right_middle_joint_3: type revolute, parent right_middle_link_2, child right_middle_link_3, origin xyz=0.03 0 0 rpy=0 0 0, axis 0 0 1, limit lower=0 upper=1.5707 effort=1 velocity=2
- added joint right_ring_joint_0: type revolute, parent right_palm, child right_ring_link_0, origin xyz=0.122 0.0315 0.00175 rpy=-3.1416 0 0, axis 0 0 1, limit lower=-0.349 upper=0.349 effort=1 velocity=2
- added joint right_ring_joint_1: type revolute, parent right_ring_link_0, child right_ring_link_1, origin xyz=0 0 0 rpy=-1.5708 0 0, axis 0 0 1, limit lower=0 upper=1.5707 effort=1 velocity=2
- added joint right_ring_joint_2: type revolute, parent right_ring_link_1, child right_ring_link_2, origin xyz=0.04 0 0 rpy=0 0 0, axis 0 0 1, limit lower=0 upper=1.5707 effort=1 velocity=2
- added joint right_ring_joint_3: type revolute, parent right_ring_link_2, child right_ring_link_3, origin xyz=0.03 0 0 rpy=0 0 0, axis 0 0 1, limit lower=0 upper=1.5707 effort=1 velocity=2
- added joint right_thumb_joint_0: type revolute, parent right_palm, child right_thumb_link_0, origin xyz=0.026 -0.0365 -0.00025 rpy=3.1416 0 -1.5708, axis 0 0 1, limit lower=-0.349 upper=0.349 effort=1 velocity=2
- added joint right_thumb_joint_1: type revolute, parent right_thumb_link_0, child right_thumb_link_1, origin xyz=0 0 0 rpy=-1.5708 0 0, axis 0 0 1, limit lower=0 upper=1.5707 effort=1 velocity=2
- added joint right_thumb_joint_2: type revolute, parent right_thumb_link_1, child right_thumb_link_2, origin xyz=0.039999 0.009 -0.0215 rpy=-1.5708 0.261799388 0, axis 0 0 1, limit lower=0 upper=1.5707 effort=1 velocity=2
- added joint right_thumb_joint_3: type revolute, parent right_thumb_link_2, child right_thumb_link_3, origin xyz=0.063268 -0.016953 0 rpy=0 0 0, axis 0 0 1, limit lower=0 upper=1.5707 effort=1 velocity=2

File: robot_simulation_ws/src/bullet_simulation_pkg/urdf/plane.urdf (robot description, URDF)
Before this commit: robot plane, 1 links, 0 joints
Links:
- link planeLink: geometry collision box size=200 200 10; visual mesh filename=package://bullet_simulation_pkg/meshes/plane100.obj scale=1 1 1

File: robot_simulation_ws/src/bullet_simulation_pkg/urdf/table.urdf (robot description, URDF)
Before this commit: robot table.urdf, 1 links, 0 joints
Links:
- link baseLink: geometry collision box size=1.5 1 0.05; visual mesh filename=package://bullet_simulation_pkg/meshes/table.obj scale=0.1 0.1 0.58
